File: eagle/board.brd (EAGLE design)
At the start: 64 x 49 mm, 31 parts

Commit message: pcb update
Parts:
- moved JP5 3.00 mm to (30.0, 5.50)
- moved JP10 2.55 mm to (44.5, 15.5)
- moved JP12 2.55 mm to (43.9, 41.1)
- moved JP6 2.55 mm to (51.0, 12.5)
- moved JP7 2.55 mm to (54.0, 12.5)
- moved JP8 2.55 mm to (44.0, 33.0)
- moved JP9 2.55 mm to (44.0, 24.0)
- moved R1 2.55 mm to (58.0, 32.5)
- moved R2 2.55 mm to (58.0, 24.5)
- moved R3 2.55 mm to (58.0, 41.0)
- moved R5 2.55 mm to (58.0, 15.5)
- moved S1 2.55 mm to (51.0, 35.0)
- moved S2 2.55 mm to (51.0, 26.5)
- moved S3 2.55 mm to (51.0, 18.0)
- moved S4 2.55 mm to (51.0, 43.5)
Routing:
- net BUT3: track 6.37 -> 7.31 mm
Other:
- board size 64 x 49 mm -> 61.5 x 49 mm

Commit message: pcb update
Parts:
- moved MOTOR2 8.30 mm to (11.3, 7.37)
- moved MOTOR1 8.00 mm to (11.3, 17.4)
- moved MOT1 1.65 mm to (17.5, 18.0)
- moved BATTERY 1.50 mm to (18.4, 45.6)
- moved C1 1.50 mm to (18.8, 39.8)
- moved C2 1.50 mm to (18.8, 42.5)
- moved MOT2 1.50 mm to (17.4, 8.00)
- moved R4 1.50 mm to (17.5, 30.0)
Routing:
- net MOT2-OUT2: track 9.90 -> 2.93 mm
- net MOT2-OUT1: track 9.73 -> 2.93 mm
- net MOT1-OUT2: track 9.38 -> 3.03 mm
- net MOT1-OUT1: track 9.38 -> 3.03 mm
- net GND: track 6.26 -> 3.86 mm
- net MOT1-2: track 4.74 -> 3.16 mm
- net N$3: track 6.06 -> 7.56 mm
- net VIN: track 53.7 -> 55.1 mm
- net 5V: track 39.0 -> 37.7 mm
- net MOT2-1: track 4.92 -> 3.68 mm
- net MOT2-2: track 5.59 -> 4.72 mm
- net MOT1-1: track 5.14 -> 4.27 mm
Other:
- board size 61.5 x 49 mm -> 57.5 x 49 mm

Commit message: added new picture
Parts:
- moved JP10 12.4 mm to (36.0, 6.50)
- moved JP12 12.4 mm to (35.4, 32.1)
- moved JP6 12.4 mm to (42.5, 3.50)
- moved JP7 12.4 mm to (45.5, 3.50)
- moved JP8 12.4 mm to (35.5, 24.0)
- moved JP9 12.4 mm to (35.5, 15.0)
- moved R1 12.4 mm to (49.5, 23.5)
- moved R2 12.4 mm to (49.5, 15.5)
- moved R3 12.4 mm to (49.5, 32.0)
- moved R5 12.4 mm to (49.5, 6.50)
- moved S1 12.4 mm to (42.5, 26.0)
- moved S2 12.4 mm to (42.5, 17.5)
- moved S3 12.4 mm to (42.5, 9.00)
- moved S4 12.4 mm to (42.5, 34.5)
- moved ARD 4.27 mm to (21.0, 2.50)
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Other:
- board size 57.5 x 49 mm -> 53 x 50 mm
