File: eagle/board.sch (EAGLE design)
At the start: 31 parts

Commit message: pcb update
Other:
- moved on the sheet: BATTERY, C1, C2, MOTOR1, MOTOR2, PIEZO, R1, R2, R3, R5, S1, S2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

Commit message: pcb update
Parts:
- removed JP11, JP5: (no value), pinhead:PINHD-1X1
- added J5V, JGND: (no value), pinhead:PINHD-1X1
- renumbered JP10 to JP3', JP12 to JP4', JP6 to J5V', JP7 to JGND', JP8 to JP1', JP9 to JP2'
Connections:
- net 5V: now also J5V.1; no longer JP1.1
- net BUT1: now also JP1.1; no longer JP3.1
- net BUT2: now also JP2.1; no longer JP4.1
- net BUT3: now also JP3.1; no longer JP5.1
- net BUT4: now also JP4.1; no longer JP11.1
- net GND: now also JGND.1; no longer JP2.1
Other:
- moved on the sheet: JP1, JP2, JP3, JP4
Changed lines of the file:
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@@
 <part name="R2" library="fab" deviceset="RES-US" device="1206FAB" value="10k"/>
 <part name="R5" library="fab" deviceset="RES-US" device="1206FAB" value="10k"/>
+<part name="J5V" library="pinhead" deviceset="PINHD-1X1" device=""/>
+<part name="JGND" library="pinhead" deviceset="PINHD-1X1" device=""/>
 <part name="JP1" library="pinhead" deviceset="PINHD-1X1" device=""/>
 <part name="JP2" library="pinhead" deviceset="PINHD-1X1" device=""/>
 <part name="JP3" library="pinhead" deviceset="PINHD-1X1" device=""/>
+<part name="J5V'" library="pinhead" deviceset="PINHD-1X1" device=""/>
+<part name="JGND'" library="pinhead" deviceset="PINHD-1X1" device=""/>
+<part name="JP1'" library="pinhead" deviceset="PINHD-1X1" device=""/>
+<part name="JP2'" library="pinhead" deviceset="PINHD-1X1" device=""/>
+<part name="JP3'" library="pinhead" deviceset="PINHD-1X1" device=""/>
 <part name="JP4" library="pinhead" deviceset="PINHD-1X1" device=""/>
-<part name="JP5" library="pinhead" deviceset="PINHD-1X1" device=""/>
-<part name="JP6" library="pinhead" deviceset="PINHD-1X1" device=""/>
-<part name="JP7" library="pinhead" deviceset="PINHD-1X1" device=""/>
-<part name="JP8" library="pinhead" deviceset="PINHD-1X1" device=""/>
-<part name="JP9" library="pinhead" deviceset="PINHD-1X1" device=""/>
-<part name="JP10" library="pinhead" deviceset="PINHD-1X1" device=""/>
-<part name="JP11" library="pinhead" deviceset="PINHD-1X1" device=""/>
-<part name="JP12" library="pinhead" deviceset="PINHD-1X1" device=""/>
+<part name="JP4'" library="pinhead" deviceset="PINHD-1X1" device=""/>
 <part name="S4" library="fab" deviceset="6MM_SWITCH" device="6MM_SWITCH"/>
 <part name="R3" library="fab" deviceset="RES-US" device="1206FAB" value="10k"/>
@@
 <instance part="R2" gate="G$1" x="284.48" y="66.04"/>
 <instance part="R5" gate="G$1" x="284.48" y="53.34"/>
-<instance part="JP1" gate="G$1" x="203.2" y="83.82"/>
-<instance part="JP2" gate="G$1" x="203.2" y="73.66"/>
-<instance part="JP3" gate="G$1" x="203.2" y="63.5"/>
-<instance part="JP4" gate="G$1" x="203.2" y="53.34"/>
-<instance part="JP5" gate="G$1" x="203.2" y="43.18"/>
-<instance part="JP6" gate="G$1" x="213.36" y="83.82" rot="R180"/>
-<instance part="JP7" gate="G$1" x="213.36" y="73.66" rot="R180"/>
-<instance part="JP8" gate="G$1" x="213.36" y="63.5" rot="R180"/>
-<instance part="JP9" gate="G$1" x="213.36" y="53.34" rot="R180"/>
-<instance part="JP10" gate="G$1" x="213.36" y="43.18" rot="R180"/>
-<instance part="JP11" gate="G$1" x="203.2" y="33.02"/>
-<instance part="JP12" gate="G$1" x="213.36" y="33.02" rot="R180"/>
+<instance part="J5V" gate="G$1" x="203.2" y="83.82"/>
+<instance part="JGND" gate="G$1" x="203.2" y="73.66"/>
+<instance part="JP1" gate="G$1" x="203.2" y="63.5"/>
+<instance part="JP2" gate="G$1" x="203.2" y="53.34"/>
+<instance part="JP3" gate="G$1" x="203.2" y="43.18"/>
+<instance part="J5V'" gate="G$1" x="213.36" y="83.82" rot="R180"/>
+<instance part="JGND'" gate="G$1" x="213.36" y="73.66" rot="R180"/>
+<instance part="JP1'" gate="G$1" x="213.36" y="63.5" rot="R180"/>
+<instance part="JP2'" gate="G$1" x="213.36" y="53.34" rot="R180"/>
+<instance part="JP3'" gate="G$1" x="213.36" y="43.18" rot="R180"/>
+<instance part="JP4" gate="G$1" x="203.2" y="33.02"/>
+<instance part="JP4'" gate="G$1" x="213.36" y="33.02" rot="R180"/>
 <instance part="S4" gate="2" x="269.24" y="40.64" rot="R270"/>
 <instance part="R3" gate="G$1" x="284.48" y="38.1"/>
@@
 </segment>
 <segment>
-<pinref part="JP3" gate="G$1" pin="1"/>
+<pinref part="JP1" gate="G$1" pin="1"/>
 <wire x1="185.42" y1="63.5" x2="200.66" y2="63.5" width="0.1524" layer="91"/>
 <label x="185.42" y="63.5" size="1.778" layer="95" rot="R180" xref="yes"/>
@@
 </segment>
 <segment>
-<pinref part="JP4" gate="G$1" pin="1"/>
+<pinref part="JP2" gate="G$1" pin="1"/>
 <wire x1="185.42" y1="53.34" x2="200.66" y2="53.34" width="0.1524" layer="91"/>
 <label x="185.42" y="53.34" size="1.778" layer="95" rot="R180" xref="yes"/>
@@
 </segment>
 <segment>
-<pinref part="JP5" gate="G$1" pin="1"/>
+<pinref part="JP3" gate="G$1" pin="1"/>
 <wire x1="185.42" y1="43.18" x2="200.66" y2="43.18" width="0.1524" layer="91"/>
 <label x="185.42" y="43.18" size="1.778" layer="95" rot="R180" xref="yes"/>
@@
 </segment>
 <segment>
-<pinref part="JP1" gate="G$1" pin="1"/>
+<pinref part="J5V" gate="G$1" pin="1"/>
 <wire x1="185.42" y1="83.82" x2="200.66" y2="83.82" width="0.1524" layer="91"/>
 <label x="185.42" y="83.82" size="1.778" layer="95" rot="R180" xref="yes"/>
@@
 </segment>
 <segment>
-<pinref part="JP2" gate="G$1" pin="1"/>
+<pinref part="JGND" gate="G$1" pin="1"/>
 <wire x1="185.42" y1="73.66" x2="200.66" y2="73.66" width="0.1524" layer="91"/>
 <label x="185.42" y="73.66" size="1.778" layer="95" rot="R180" xref="yes"/>
@@
 </segment>
 <segment>
-<pinref part="JP6" gate="G$1" pin="1"/>
+<pinref part="J5V'" gate="G$1" pin="1"/>
 <wire x1="215.9" y1="83.82" x2="231.14" y2="83.82" width="0.1524" layer="91"/>
 <label x="231.14" y="83.82" size="1.778" layer="95" xref="yes"/>
@@
 </segment>
 <segment>
-<pinref part="JP8" gate="G$1" pin="1"/>
+<pinref part="JP1'" gate="G$1" pin="1"/>
 <wire x1="215.9" y1="63.5" x2="231.14" y2="63.5" width="0.1524" layer="91"/>
 <label x="231.14" y="63.5" size="1.778" layer="95" xref="yes"/>
@@
 </segment>
 <segment>
-<pinref part="JP9" gate="G$1" pin="1"/>
+<pinref part="JP2'" gate="G$1" pin="1"/>
 <wire x1="215.9" y1="53.34" x2="231.14" y2="53.34" width="0.1524" layer="91"/>
 <label x="231.14" y="53.34" size="1.778" layer="95" xref="yes"/>
@@
 </segment>
 <segment>
-<pinref part="JP10" gate="G$1" pin="1"/>
+<pinref part="JP3'" gate="G$1" pin="1"/>
 <wire x1="215.9" y1="43.18" x2="231.14" y2="43.18" width="0.1524" layer="91"/>
 <label x="231.14" y="43.18" size="1.778" layer="95" xref="yes"/>
@@
 </segment>
 <segment>
-<pinref part="JP7" gate="G$1" pin="1"/>
+<pinref part="JGND'" gate="G$1" pin="1"/>
 <wire x1="215.9" y1="73.66" x2="231.14" y2="73.66" width="0.1524" layer="91"/>
 <label x="231.14" y="73.66" size="1.778" layer="95" xref="yes"/>
@@
 <net name="BUT4" class="0">
 <segment>
-<pinref part="JP11" gate="G$1" pin="1"/>
+<pinref part="JP4" gate="G$1" pin="1"/>
 <wire x1="185.42" y1="33.02" x2="200.66" y2="33.02" width="0.1524" layer="91"/>
 <label x="185.42" y="33.02" size="1.778" layer="95" rot="R180" xref="yes"/>
@@
 <segment>
 <label x="231.14" y="33.02" size="1.778" layer="95" xref="yes"/>
-<pinref part="JP12" gate="G$1" pin="1"/>
+<pinref part="JP4'" gate="G$1" pin="1"/>
 <wire x1="215.9" y1="33.02" x2="231.14" y2="33.02" width="0.1524" layer="91"/>
 </segment>
@@
 </sheet>
 </sheets>
-<errors>
-</errors>
 </schematic>
 </drawing>
